Commit message: gripper working but phone not

File: robosuite/models/assets/robots/ur3e_with_gripper/ur3e.urdf (robot description, URDF)
Before this commit: robot ur3e_robot, 11 links, 10 joints
Links:
- link base_link_inertia: geometry collision mesh filename=/home/biorobotics-ms/d3_plan_ws/src/fmauch_universal_robot/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; visual mesh filename=/home/biorobotics-ms/d3_plan_ws/src/fmauch_universal_robot/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
- link forearm_link: geometry collision mesh filename=/home/biorobotics-ms/d3_plan_ws/src/fmauch_universal_robot/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; visual mesh filename=/home/biorobotics-ms/d3_plan_ws/src/fmauch_universal_robot/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
- link shoulder_link: geometry collision mesh filename=/home/biorobotics-ms/d3_plan_ws/src/fmauch_universal_robot/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; visual mesh filename=/home/biorobotics-ms/d3_plan_ws/src/fmauch_universal_robot/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
- link upper_arm_link: geometry collision mesh filename=/home/biorobotics-ms/d3_plan_ws/src/fmauch_universal_robot/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; visual mesh filename=/home/biorobotics-ms/d3_plan_ws/src/fmauch_universal_robot/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
- link wrist_1_link: geometry collision mesh filename=/home/biorobotics-ms/d3_plan_ws/src/fmauch_universal_robot/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; visual mesh filename=/home/biorobotics-ms/d3_plan_ws/src/fmauch_universal_robot/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
- link wrist_2_link: geometry collision mesh filename=/home/biorobotics-ms/d3_plan_ws/src/fmauch_universal_robot/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; visual mesh filename=/home/biorobotics-ms/d3_plan_ws/src/fmauch_universal_robot/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
- link wrist_3_link: geometry collision mesh filename=/home/biorobotics-ms/d3_plan_ws/src/fmauch_universal_robot/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; visual mesh filename=/home/biorobotics-ms/d3_plan_ws/src/fmauch_universal_robot/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
